File: power/power.sch (KiCad schematic (older format))
At the start: 7 parts, among them J1 Conn_01x08_Male, J2 Conn_01x08_Male, J3 Jack-DC

Commit message: Ready
Parts:
- removed J1, J2: Conn_01x08_Male, Connector_PinHeader_2.54mm:PinHeader_1x08_P2.54mm_Vertical, symbol Connector:Conn_01x08_Male
- added J1, J2, J4, J5, J6, J7, J8, J9: Conn_01x06_Male, MyLib:PinHeader_1x06_P2.54mm_Vertical_BigHoles, symbol Connector:Conn_01x06_Male
- added RN1, RN2: R_Network06, Resistor_THT:R_Array_SIP7, symbol Device:R_Network06
Connections:
- wire segments 20 -> 72
