File: r-2r/r-2r.sch (KiCad schematic (older format))
At the start: 25 parts, among them J1 D7, J2 D6, J3 D5, J4 D4, J5 D3, J6 D2, J7 D1, J8 D0, J9 Out

Commit message: R-2R pcb
Parts:
- added J10: Gnd, Connector_PinHeader_2.54mm:PinHeader_1x01_P2.54mm_Vertical, symbol Connector:Conn_01x01_Male
- J1, J2, J3, J4, J5, J6, J7, J8, J9: footprint (none) -> Connector_PinHeader_2.54mm:PinHeader_1x01_P2.54mm_Vertical
- R1, R10, R11, R12, R13, R14, R15, R16, R2, R3, R4, R5, R6, R7, R8, R9: footprint (none) -> Resistor_THT:R_Axial_DIN0204_L3.6mm_D1.6mm_P7.62mm_Horizontal
Connections:
- wire segments 33 -> 35
Changed lines of the file:
@@
 EESchema Schematic File Version 4
+LIBS:r-2r-cache
 EELAYER 26 0
 EELAYER END
@@
 F 0 "R1" V 3093 1650 50  0000 C CNN
 F 1 "2k" V 3184 1650 50  0000 C CNN
-F 2 "" V 3230 1650 50  0001 C CNN
+F 2 "Resistor_THT:R_Axial_DIN0204_L3.6mm_D1.6mm_P7.62mm_Horizontal" V 3230 1650 50  0001 C CNN
 F 3 "~" H 3300 1650 50  0001 C CNN
 	1    3300 1650
@@
 F 0 "R9" H 3620 1946 50  0000 L CNN
 F 1 "1k" H 3620 1855 50  0000 L CNN
-F 2 "" V 3480 1900 50  0001 C CNN
+F 2 "Resistor_THT:R_Axial_DIN0204_L3.6mm_D1.6mm_P7.62mm_Horizontal" V 3480 1900 50  0001 C CNN
 F 3 "~" H 3550 1900 50  0001 C CNN
 	1    3550 1900
@@
 F 0 "R2" V 3093 2150 50  0000 C CNN
 F 1 "2k" V 3184 2150 50  0000 C CNN
-F 2 "" V 3230 2150 50  0001 C CNN
+F 2 "Resistor_THT:R_Axial_DIN0204_L3.6mm_D1.6mm_P7.62mm_Horizontal" V 3230 2150 50  0001 C CNN
 F 3 "~" H 3300 2150 50  0001 C CNN
 	1    3300 2150
@@
 F 0 "R10" H 3620 2446 50  0000 L CNN
 F 1 "1k" H 3620 2355 50  0000 L CNN
-F 2 "" V 3480 2400 50  0001 C CNN
+F 2 "Resistor_THT:R_Axial_DIN0204_L3.6mm_D1.6mm_P7.62mm_Horizontal" V 3480 2400 50  0001 C CNN
 F 3 "~" H 3550 2400 50  0001 C CNN
 	1    3550 2400
@@
 F 0 "R13" H 3620 3946 50  0000 L CNN
 F 1 "1k" H 3620 3855 50  0000 L CNN
-F 2 "" V 3480 3900 50  0001 C CNN
+F 2 "Resistor_THT:R_Axial_DIN0204_L3.6mm_D1.6mm_P7.62mm_Horizontal" V 3480 3900 50  0001 C CNN
 F 3 "~" H 3550 3900 50  0001 C CNN
 	1    3550 3900
@@
 F 0 "R6" V 3093 4150 50  0000 C CNN
 F 1 "2k" V 3184 4150 50  0000 C CNN
-F 2 "" V 3230 4150 50  0001 C CNN
+F 2 "Resistor_THT:R_Axial_DIN0204_L3.6mm_D1.6mm_P7.62mm_Horizontal" V 3230 4150 50  0001 C CNN
 F 3 "~" H 3300 4150 50  0001 C CNN
 	1    3300 4150
@@
 F 0 "R14" H 3620 4446 50  0000 L CNN
 F 1 "1k" H 3620 4355 50  0000 L CNN
-F 2 "" V 3480 4400 50  0001 C CNN
+F 2 "Resistor_THT:R_Axial_DIN0204_L3.6mm_D1.6mm_P7.62mm_Horizontal" V 3480 4400 50  0001 C CNN
 F 3 "~" H 3550 4400 50  0001 C CNN
 	1    3550 4400
@@
 F 0 "R7" V 3093 4650 50  0000 C CNN
 F 1 "2k" V 3184 4650 50  0000 C CNN
-F 2 "" V 3230 4650 50  0001 C CNN
+F 2 "Resistor_THT:R_Axial_DIN0204_L3.6mm_D1.6mm_P7.62mm_Horizontal" V 3230 4650 50  0001 C CNN
 F 3 "~" H 3300 4650 50  0001 C CNN
 	1    3300 4650
@@
 F 0 "R15" H 3620 4946 50  0000 L CNN
 F 1 "1k" H 3620 4855 50  0000 L CNN
-F 2 "" V 3480 4900 50  0001 C CNN
+F 2 "Resistor_THT:R_Axial_DIN0204_L3.6mm_D1.6mm_P7.62mm_Horizontal" V 3480 4900 50  0001 C CNN
 F 3 "~" H 3550 4900 50  0001 C CNN
 	1    3550 4900
@@
 F 0 "R3" V 3093 2650 50  0000 C CNN
 F 1 "2k" V 3184 2650 50  0000 C CNN
-F 2 "" V 3230 2650 50  0001 C CNN
+F 2 "Resistor_THT:R_Axial_DIN0204_L3.6mm_D1.6mm_P7.62mm_Horizontal" V 3230 2650 50  0001 C CNN
 F 3 "~" H 3300 2650 50  0001 C CNN
 	1    3300 2650
@@
 F 0 "R11" H 3620 2946 50  0000 L CNN
 F 1 "1k" H 3620 2855 50  0000 L CNN
-F 2 "" V 3480 2900 50  0001 C CNN
+F 2 "Resistor_THT:R_Axial_DIN0204_L3.6mm_D1.6mm_P7.62mm_Horizontal" V 3480 2900 50  0001 C CNN
 F 3 "~" H 3550 2900 50  0001 C CNN
 	1    3550 2900
@@
 F 0 "R4" V 3093 3150 50  0000 C CNN
 F 1 "2k" V 3184 3150 50  0000 C CNN
-F 2 "" V 3230 3150 50  0001 C CNN
+F 2 "Resistor_THT:R_Axial_DIN0204_L3.6mm_D1.6mm_P7.62mm_Horizontal" V 3230 3150 50  0001 C CNN
 F 3 "~" H 3300 3150 50  0001 C CNN
 	1    3300 3150
@@
 F 0 "R12" H 3620 3446 50  0000 L CNN
 F 1 "1k" H 3620 3355 50  0000 L CNN
-F 2 "" V 3480 3400 50  0001 C CNN
+F 2 "Resistor_THT:R_Axial_DIN0204_L3.6mm_D1.6mm_P7.62mm_Horizontal" V 3480 3400 50  0001 C CNN
 F 3 "~" H 3550 3400 50  0001 C CNN
 	1    3550 3400
@@
 F 0 "R5" V 3093 3650 50  0000 C CNN
 F 1 "2k" V 3184 3650 50  0000 C CNN
-F 2 "" V 3230 3650 50  0001 C CNN
+F 2 "Resistor_THT:R_Axial_DIN0204_L3.6mm_D1.6mm_P7.62mm_Horizontal" V 3230 3650 50  0001 C CNN
 F 3 "~" H 3300 3650 50  0001 C CNN
 	1    3300 3650
@@
 F 0 "R8" V 3093 5150 50  0000 C CNN
 F 1 "2k" V 3184 5150 50  0000 C CNN
-F 2 "" V 3230 5150 50  0001 C CNN
+F 2 "Resistor_THT:R_Axial_DIN0204_L3.6mm_D1.6mm_P7.62mm_Horizontal" V 3230 5150 50  0001 C CNN
 F 3 "~" H 3300 5150 50  0001 C CNN
 	1    3300 5150
@@
 F 0 "R16" H 3620 5446 50  0000 L CNN
 F 1 "2k" H 3620 5355 50  0000 L CNN
-F 2 "" V 3480 5400 50  0001 C CNN
+F 2 "Resistor_THT:R_Axial_DIN0204_L3.6mm_D1.6mm_P7.62mm_Horizontal" V 3480 5400 50  0001 C CNN
 F 3 "~" H 3550 5400 50  0001 C CNN
 	1    3550 5400
@@
 F 0 "J1" H 2706 1828 50  0000 C CNN
 F 1 "D7" H 2706 1737 50  0000 C CNN
-F 2 "" H 2600 1650 50  0001 C CNN
+F 2 "Connector_PinHeader_2.54mm:PinHeader_1x01_P2.54mm_Vertical" H 2600 1650 50  0001 C CNN
 F 3 "~" H 2600 1650 50  0001 C CNN
 	1    2600 1650
@@
 F 0 "J2" H 2706 2328 50  0000 C CNN
 F 1 "D6" H 2706 2237 50  0000 C CNN
-F 2 "" H 2600 2150 50  0001 C CNN
+F 2 "Connector_PinHeader_2.54mm:PinHeader_1x01_P2.54mm_Vertical" H 2600 2150 50  0001 C CNN
 F 3 "~" H 2600 2150 50  0001 C CNN
 	1    2600 2150
@@
 F 0 "J3" H 2706 2828 50  0000 C CNN
 F 1 "D5" H 2706 2737 50  0000 C CNN
-F 2 "" H 2600 2650 50  0001 C CNN
+F 2 "Connector_PinHeader_2.54mm:PinHeader_1x01_P2.54mm_Vertical" H 2600 2650 50  0001 C CNN
 F 3 "~" H 2600 2650 50  0001 C CNN
 	1    2600 2650
@@
 F 0 "J4" H 2706 3328 50  0000 C CNN
 F 1 "D4" H 2706 3237 50  0000 C CNN
-F 2 "" H 2600 3150 50  0001 C CNN
+F 2 "Connector_PinHeader_2.54mm:PinHeader_1x01_P2.54mm_Vertical" H 2600 3150 50  0001 C CNN
 F 3 "~" H 2600 3150 50  0001 C CNN
 	1    2600 3150
@@
 F 0 "J5" H 2706 3828 50  0000 C CNN
 F 1 "D3" H 2706 3737 50  0000 C CNN
-F 2 "" H 2600 3650 50  0001 C CNN
+F 2 "Connector_PinHeader_2.54mm:PinHeader_1x01_P2.54mm_Vertical" H 2600 3650 50  0001 C CNN
 F 3 "~" H 2600 3650 50  0001 C CNN
 	1    2600 3650
@@
 F 0 "J6" H 2706 4328 50  0000 C CNN
 F 1 "D2" H 2706 4237 50  0000 C CNN
-F 2 "" H 2600 4150 50  0001 C CNN
+F 2 "Connector_PinHeader_2.54mm:PinHeader_1x01_P2.54mm_Vertical" H 2600 4150 50  0001 C CNN
 F 3 "~" H 2600 4150 50  0001 C CNN
 	1    2600 4150
@@
 F 0 "J7" H 2706 4828 50  0000 C CNN
 F 1 "D1" H 2706 4737 50  0000 C CNN
-F 2 "" H 2600 4650 50  0001 C CNN
+F 2 "Connector_PinHeader_2.54mm:PinHeader_1x01_P2.54mm_Vertical" H 2600 4650 50  0001 C CNN
 F 3 "~" H 2600 4650 50  0001 C CNN
 	1    2600 4650
@@
 F 0 "J8" H 2706 5328 50  0000 C CNN
 F 1 "D0" H 2706 5237 50  0000 C CNN
-F 2 "" H 2600 5150 50  0001 C CNN
+F 2 "Connector_PinHeader_2.54mm:PinHeader_1x01_P2.54mm_Vertical" H 2600 5150 50  0001 C CNN
 F 3 "~" H 2600 5150 50  0001 C CNN
 	1    2600 5150
@@
 	2800 5150 3150 5150
 Wire Wire Line
-	3550 5550 3550 5750
+	3550 5550 3550 5600
 Wire Wire Line
 	3550 5050 3550 5150
@@
 F 0 "J9" H 3873 1673 50  0000 R CNN
 F 1 "Out" H 3873 1582 50  0000 R CNN
-F 2 "" H 3900 1650 50  0001 C CNN
+F 2 "Connector_PinHeader_2.54mm:PinHeader_1x01_P2.54mm_Vertical" H 3900 1650 50  0001 C CNN
 F 3 "~" H 3900 1650 50  0001 C CNN
 	1    3900 1650
@@
 	3700 1650 3550 1650
 Connection ~ 3550 1650
+$Comp
+L Connector:Conn_01x01_Male J10
+U 1 1 5D2E3396
+P 3900 5600
+F 0 "J10" H 3873 5623 50  0000 R CNN
+F 1 "Gnd" H 3873 5532 50  0000 R CNN
+F 2 "Connector_PinHeader_2.54mm:PinHeader_1x01_P2.54mm_Vertical" H 3900 5600 50  0001 C CNN
+F 3 "~" H 3900 5600 50  0001 C CNN
+	1    3900 5600
+	-1   0    0    -1
+$EndComp
+Wire Wire Line
+	3550 5600 3700 5600
+Connection ~ 3550 5600
+Wire Wire Line
+	3550 5600 3550 5750
 $EndSCHEMATC

Commit message: Add mounting holes
Parts:
- added MH1, MH2, MH3, MH4: MountingHole, MountingHole:MountingHole_3.2mm_M3_Pad_Via, symbol Mechanical:MountingHole
Changed lines of the file:
@@
 Wire Wire Line
 	3550 5600 3550 5750
+$Comp
+L Mechanical:MountingHole MH1
+U 1 1 5D2F69F0
+P 5500 1600
+F 0 "MH1" H 5600 1646 50  0000 L CNN
+F 1 "MountingHole" H 5600 1555 50  0000 L CNN
+F 2 "MountingHole:MountingHole_3.2mm_M3_Pad_Via" H 5500 1600 50  0001 C CNN
+F 3 "~" H 5500 1600 50  0001 C CNN
+	1    5500 1600
+	1    0    0    -1
+$EndComp
+$Comp
+L Mechanical:MountingHole MH2
+U 1 1 5D2F6A76
+P 5500 1900
+F 0 "MH2" H 5600 1946 50  0000 L CNN
+F 1 "MountingHole" H 5600 1855 50  0000 L CNN
+F 2 "MountingHole:MountingHole_3.2mm_M3_Pad_Via" H 5500 1900 50  0001 C CNN
+F 3 "~" H 5500 1900 50  0001 C CNN
+	1    5500 1900
+	1    0    0    -1
+$EndComp
+$Comp
+L Mechanical:MountingHole MH3
+U 1 1 5D2F6AD6
+P 5500 2200
+F 0 "MH3" H 5600 2246 50  0000 L CNN
+F 1 "MountingHole" H 5600 2155 50  0000 L CNN
+F 2 "MountingHole:MountingHole_3.2mm_M3_Pad_Via" H 5500 2200 50  0001 C CNN
+F 3 "~" H 5500 2200 50  0001 C CNN
+	1    5500 2200
+	1    0    0    -1
+$EndComp
+$Comp
+L Mechanical:MountingHole MH4
+U 1 1 5D2F6B38
+P 5500 2500
+F 0 "MH4" H 5600 2546 50  0000 L CNN
+F 1 "MountingHole" H 5600 2455 50  0000 L CNN
+F 2 "MountingHole:MountingHole_3.2mm_M3_Pad_Via" H 5500 2500 50  0001 C CNN
+F 3 "~" H 5500 2500 50  0001 C CNN
+	1    5500 2500
+	1    0    0    -1
+$EndComp
 $EndSCHEMATC
